Commit message: added hubcaps

File: urdf/robot.urdf (robot description, URDF)
Before this commit: robot robot, 3 links, 2 joints
Links:
- link link_left_wheel: geometry collision box size=0.6 0.05 0.02; collision cylinder length=0.12 radius=0.08
- link link_right_wheel: geometry collision box size=0.6 0.05 0.02; collision cylinder length=0.12 radius=0.08

Commit message: added caster wheel, needs tuning

File: urdf/robot.urdf (robot description, URDF)
Before this commit: robot robot, 3 links, 2 joints
Links:
- added link caster_wheel, mass 10; collision sphere radius=0.125; collision sphere radius=0.25
Joints:
- added joint caster_wheel: type fixed, parent link_chassis, child caster_wheel, origin xyz=-0.5 -0.65 0 rpy=0 0 0, axis 0 1 0, limit effort=10000 velocity=1000

Commit message: caster wheel placement tuned

File: urdf/robot.urdf (robot description, URDF)
Before this commit: robot robot, 4 links, 3 joints
Joints:
- joint caster_wheel: origin xyz=-0.5 -0.65 0 rpy=0 0 0 -> xyz=0.75 0 -0.125 rpy=0 0 0

Commit message: meshes for chassis + wheel tires, tuned geometry

File: urdf/robot.urdf (robot description, URDF)
Before this commit: robot robot, 4 links, 3 joints
Links:
- link link_chassis: geometry collision box size=2 1.3 0.4; visual mesh filename=package://robot_description/meshes/chassis.stl
- link link_left_wheel: geometry collision box size=0.6 0.05 0.02; collision cylinder length=0.12 radius=0.08
- link link_right_wheel: geometry collision box size=0.6 0.05 0.02; collision cylinder length=0.12 radius=0.08

Commit message: gazebo tags for colors and friction in URDF file

File: urdf/robot.urdf (robot description, URDF)
Before this commit: robot robot, 4 links, 3 joints
Links:
- removed link caster_wheel
- added link link_caster_wheel, mass 1; collision sphere radius=0.125; collision sphere radius=0.25
Joints:
- removed joint caster_wheel
- added joint joint_chassis_caster_wheel: type fixed, parent link_chassis, child link_caster_wheel, origin xyz=0.75 0 -0.125 rpy=0 0 0
