Commit message: replace urdf with xacro

File: urdf/robot.xacro (robot description, xacro)
@@ -1,82 +1,11 @@
 <?xml version="1.0" ?>
-<robot name="robot">
-    <!-- Gazebo simulator tags -->
-    <gazebo reference="link_chassis">
-        <material>Gazebo/Blue</material>
-    </gazebo>
-    <gazebo reference="link_caster_wheel">
-        <material>Gazebo/Grey</material>
-        <mu1>0.0</mu1>
-        <mu2>0.0</mu2>
-    </gazebo>
-    <gazebo reference="link_left_wheel">
-        <material>Gazebo/Black</material>
-        <mu1>1.0</mu1>
-        <mu2>1.0</mu2>
-    </gazebo>
-    <gazebo reference="link_right_wheel">
-        <material>Gazebo/Black</material>
-        <mu1>1.0</mu1>
-        <mu2>1.0</mu2>
-    </gazebo>
-    <gazebo reference="joint_chassis_caster_wheel">
-        <preserveFixedJoint>true</preserveFixedJoint> <!-- Don't fuse to chassis -->
-    </gazebo>
-    <gazebo>
-        <plugin filename="libgazebo_ros_diff_drive.so" name="differential_drive_controller">
-            <alwaysOn>true</alwaysOn>
-            <updateRate>20</updateRate>
-            <leftJoint>joint_chassis_left_wheel</leftJoint>
-            <rightJoint>joint_chassis_right_wheel</rightJoint>
-            <wheelSeparation>1.66</wheelSeparation> <!-- TODO: update for mesh tires -->
-            <wheelDiameter>0.8</wheelDiameter> <!-- TODO: check if this is true -->
-            <torque>10</torque>
-            <commandTopic>cmd_vel</commandTopic>
-            <odometryTopic>odom</odometryTopic>
-            <odometryFrame>odom</odometryFrame>
-            <robotBaseFrame>link_chassis</robotBaseFrame>
-        </plugin>
-    </gazebo>
-        <gazebo reference="joint_laser_scan_chassis">
-        <preserveFixedJoint>true</preserveFixedJoint> <!-- Don't fuse to chassis -->
-    </gazebo>
-    <gazebo reference="link_laser_scan">
-        <material>Gazebo/DarkGrey</material>
-    </gazebo>
-    <gazebo reference="link_laser_scan">
-        <sensor type="ray" name="head_hokuyo_sensor">
-            <pose>0 0 0 0 0 0</pose>
-            <visualize>true</visualize> <!-- Simulate rays -->
-            <update_rate>20</update_rate>
-            <ray>
-                <scan>
-                    <horizontal>
-                        <samples>720</samples>
-                        <resolution>1</resolution>
-                        <min_angle>-1.570796</min_angle> <!-- ~ -90 deg -->
-                        <max_angle>1.570796</max_angle> <!-- ~ 90 deg -->
-                    </horizontal>
-                </scan>
-                <range> <!-- Should be outside "devide" cylinder! -->
-                    <min>0.20</min>
-                    <max>10.0</max>
-                    <resolution>0.01</resolution>
-                </range>
-                <noise>
-                    <type>gaussian</type>
-                    <mean>0.0</mean>
-                    <stddev>0.01</stddev>
-                </noise>
-            </ray>
-            <plugin name="gazebo_ros_head_hokuyo_controller" filename="libgazebo_ros_laser.so">
-                <topicName>/laser/scan</topicName>
-                <frameName>sensor_laser</frameName>
-            </plugin>
-        </sensor>
-    </gazebo>
+<robot name="robot" xmlns:xacro="http://www.ros.org/wiki/xacro">
+    <xacro:include filename="$(find robot_description)/urdf/robot.gazebo" />
+    <!-- Parameters -->
+    <xacro:property name="chassis_mass" value="10" />
     <!-- Link - chassis -->
     <link name="link_chassis">
         <inertial>
-            <mass value="10" />
+            <mass value="${chassis_mass}" />
             <origin xyz="0 0 0.3" rpy="0 0 0" />
             <inertia ixx="1.5417" ixy="0" ixz="0" iyy="3.467" iyz="0" izz="4.742" />

Commit message: replaced half-pi radians with pi param

File: urdf/robot.xacro (robot description, xacro)
@@ -4,4 +4,5 @@
     <!-- Parameters -->
     <xacro:property name="chassis_mass" value="10" />
+    <xacro:property name="pi" value="3.1415926535" />
     <!-- Link - chassis -->
     <link name="link_chassis">
@@ -35,6 +36,6 @@
         <!-- left tire -->
         <collision>
-            <!-- <origin rpy="1.5707 0 0" xyz="0 0.18 0" /> -->
-            <origin rpy="1.5707 0 0" xyz="0 0.12 0" />
+            <!-- <origin rpy="${pi / 2} 0 0" xyz="0 0.18 0" /> -->
+            <origin rpy="${pi / 2} 0 0" xyz="0 0.12 0" />
             <geometry>
                 <cylinder length="0.12" radius="0.4"/>
@@ -42,6 +43,6 @@
         </collision>
         <visual>
-            <!-- <origin rpy="1.5707 0 0" xyz="0 0.18 0" /> -->
-            <origin rpy="1.5707 0 0" xyz="0 0.12 0" />
+            <!-- <origin rpy="${pi / 2} 0 0" xyz="0 0.18 0" /> -->
+            <origin rpy="${pi / 2} 0 0" xyz="0 0.12 0" />
             <geometry>
                 <!-- <cylinder length="0.12" radius="0.4"/> -->
@@ -54,11 +55,11 @@
         <!-- left axle -->
         <collision>
-            <origin rpy="1.5707 0 0" xyz="0 0.06 0" />
-            <geometry>
-                <cylinder length="0.12" radius="0.08"/>
-            </geometry>
-        </collision>
-        <visual>
-            <origin rpy="1.5707 0 0" xyz="0 0.06 0" />
+            <origin rpy="${pi / 2} 0 0" xyz="0 0.06 0" />
+            <geometry>
+                <cylinder length="0.12" radius="0.08"/>
+            </geometry>
+        </collision>
+        <visual>
+            <origin rpy="${pi / 2} 0 0" xyz="0 0.06 0" />
             <geometry>
                 <cylinder length="0.12" radius="0.08"/>
@@ -70,13 +71,13 @@
         <!-- left spoke -->
         <collision>
-            <!-- <origin rpy="1.5707 0 0" xyz="0 0.265 0.01" /> -->
-            <origin rpy="1.5707 0 0" xyz="0 0.12 0.01" />
-            <geometry>
-                <box size="0.6 0.05 0.02"/>
-            </geometry>
-        </collision>
-        <visual>
-            <!-- <origin rpy="1.5707 0 0" xyz="0 0.265 0.01" /> -->
-            <origin rpy="1.5707 0 0" xyz="0 0.12 0.01" />
+            <!-- <origin rpy="${pi / 2} 0 0" xyz="0 0.265 0.01" /> -->
+            <origin rpy="${pi / 2} 0 0" xyz="0 0.12 0.01" />
+            <geometry>
+                <box size="0.6 0.05 0.02"/>
+            </geometry>
+        </collision>
+        <visual>
+            <!-- <origin rpy="${pi / 2} 0 0" xyz="0 0.265 0.01" /> -->
+            <origin rpy="${pi / 2} 0 0" xyz="0 0.12 0.01" />
             <geometry>
                 <box size="0.6 0.05 0.02"/>
@@ -105,6 +106,6 @@
         </inertial>
         <collision>
-            <!-- <origin rpy="1.5707 0 0" xyz="0 -0.18 0" /> -->
-            <origin rpy="1.5707 0 0" xyz="0 -0.12 0" />
+            <!-- <origin rpy="${pi / 2} 0 0" xyz="0 -0.18 0" /> -->
+            <origin rpy="${pi / 2} 0 0" xyz="0 -0.12 0" />
             <geometry>
                 <cylinder length="0.12" radius="0.4"/>
@@ -112,6 +113,6 @@
         </collision>
         <visual>
-            <!-- <origin rpy="1.5707 0 0" xyz="0 -0.18 0" /> -->
-            <origin rpy="1.5707 0 0" xyz="0 -0.12 0" />
+            <!-- <origin rpy="${pi / 2} 0 0" xyz="0 -0.18 0" /> -->
+            <origin rpy="${pi / 2} 0 0" xyz="0 -0.12 0" />
             <geometry>
                 <!-- <cylinder length="0.12" radius="0.4"/> -->
@@ -124,11 +125,11 @@
         <!-- right axle -->
         <collision>
-            <origin rpy="1.5707 0 0" xyz="0 -0.06 0" />
-            <geometry>
-                <cylinder length="0.12" radius="0.08"/>
-            </geometry>
-        </collision>
-        <visual>
-            <origin rpy="1.5707 0 0" xyz="0 -0.06 0" />
+            <origin rpy="${pi / 2} 0 0" xyz="0 -0.06 0" />
+            <geometry>
+                <cylinder length="0.12" radius="0.08"/>
+            </geometry>
+        </collision>
+        <visual>
+            <origin rpy="${pi / 2} 0 0" xyz="0 -0.06 0" />
             <geometry>
                 <cylinder length="0.12" radius="0.08"/>
@@ -140,13 +141,13 @@
         <!-- right spoke -->
         <collision>
-            <!-- <origin rpy="1.5707 0 0" xyz="0 -0.265 0.01" /> -->
-            <origin rpy="1.5707 0 0" xyz="0 -0.12 0.01" />
-            <geometry>
-                <box size="0.6 0.05 0.02"/>
-            </geometry>
-        </collision>
-        <visual>
-            <!-- <origin rpy="1.5707 0 0" xyz="0 -0.265 0.01" /> -->
-            <origin rpy="1.5707 0 0" xyz="0 -0.12 0.01" />
+            <!-- <origin rpy="${pi / 2} 0 0" xyz="0 -0.265 0.01" /> -->
+            <origin rpy="${pi / 2} 0 0" xyz="0 -0.12 0.01" />
+            <geometry>
+                <box size="0.6 0.05 0.02"/>
+            </geometry>
+        </collision>
+        <visual>
+            <!-- <origin rpy="${pi / 2} 0 0" xyz="0 -0.265 0.01" /> -->
+            <origin rpy="${pi / 2} 0 0" xyz="0 -0.12 0.01" />
             <geometry>
                 <box size="0.6 0.05 0.02"/>

Commit message: robot controller

File: urdf/robot.xacro (robot description, xacro)
@@ -244,3 +244,45 @@
         <joint_properties damping="1.0" friction="1.0" />
     </joint>
+    <!-- Link - robot tail -->
+    <link name="link_tail">
+        <inertial>
+            <origin xyz="0 0 0" rpy="0 0 0" />
+            <mass value="0.5" />
+            <inertia ixx="0.000252666666667" ixy="0" ixz="0" iyy="0.000252666666667" iyz="0" izz="0.0005"/>
+        </inertial>
+        <visual>
+            <origin xyz="-0.2 0 0" rpy="0 ${pi/2} 0" />
+            <geometry>
+                <cylinder radius="0.05" length="0.40"/>
+            </geometry>
+            <material name="Red">
+                <color rgba="0.7 0.1 0.1 1" />
+            </material>
+        </visual>
+        <collision>
+            <origin xyz="-0.2 0 0" rpy="0 ${pi/2} 0"/>
+            <geometry>
+                <cylinder radius="0.05" length="0.40"/>
+            </geometry>
+        </collision>
+    </link>
+    <!-- Joint - chassis - robot tail-->
+    <joint name="joint_tail" type="continuous">
+        <origin rpy="0 0 0" xyz="-1 0 0" />
+        <child link="link_tail" />
+        <axis rpy="0 0 0" xyz="0 1 0" />
+        <parent link="link_chassis" />
+        <joint_properties damping="1.0" friction="1.0" />
+    </joint>
+    <!-- Transmission - joint tail-->
+    <transmission name="tran_tail">
+        <type>transmission_interface/SimpleTransmission</type>
+        <joint name="joint_tail">
+            <hardwareInterface>hardware_interface/EffortJointInterface</hardwareInterface>
+        </joint>
+        <actuator name="motor_joint_tail">
+            <hardwareInterface>hardware_interface/EffortJointInterface</hardwareInterface>
+            <mechanicalReduction>1</mechanicalReduction>
+        </actuator>
+    </transmission>
 </robot>
